File: TKL/TKL/LEDs.kicad_sch (KiCad schematic)
At the start: 89 parts, among them U1 L_TILDE, U10 L_LCTRL, U11 L_Z, U12 L_2, U13 L_F2, U14 L_W, U15 L_S, U16 L_LWIN, U17 L_X, U18 L_3, U19 L_F3, U2 L_Escape, U20 L_E, U21 L_D, U22 L_LALT, U23 L_C, U24 L_4, U25 L_F4, U26 L_R, U27 L_F, U28 L_V, U29 L_SPACE2, U3 L_TAB, U30 L_5, U31 L_F5, U32 L_T, U33 L_G, U34 L_RALT, U35 L_B, U36 L_6, U37 L_F6, U38 L_Y, U39 L_RWIN, U4 L_CAPS, U40 L_H, U41 L_N, U42 L_F7, U43 L_7, U44 L_U, U45 L_MENU, U46 L_J, U47 L_M, U48 L_F8, U49 L_8, U5 L_LSHIFT, U50 L_I, U51 L_RCTRL, U52 L_K, U53 L_COMMA, U54 L_F9, U55 L_9, U56 L_O, U57 L_LEFT, U58 L_L, U59 L_DOT, U6 L_1, U60 L_0, U61 L_F10, U62 L_P, U63 L_DOWN, U64 L_SLASH, U65 L_SEMI, U66 L_MINUS, U67 L_F11, U68 L_BRACEL, U69 L_RIGHT, U7 L_F1, U70 L_RSHIFT, U71 L_APO, U72 L_PLUS, U73 L_F12, U74 L_BRACER, U75 L_UP, U76 L_ENTER, U77 L_BACK, U78 L_PrtSc, U79 L_BCKSLSH, U8 L_Q, U80 L_INSERT, U81 L_ScrlLck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

Commit message: fixed tkl schematic
Connections:
- net GND: now also U59.3 (GND)
Changed lines of the file:
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@@
     )
   )
-  (symbol (lib_id "power:GND") (at 284.48 135.89 0) (unit 1)
+  (symbol (lib_id "power:GND") (at 284.48 137.16 0) (unit 1)
     (in_bom yes) (on_board yes) (dnp no)
-    (property "Reference" "#PWR0173" (at 284.48 142.24 0)
+    (property "Reference" "#PWR0173" (at 284.48 143.51 0)
       (effects (font (size 1.27 1.27)) hide)
     )
-    (property "Value" "GND" (at 284.607 140.2842 0)
+    (property "Value" "GND" (at 284.607 141.5542 0)
       (effects (font (size 1.27 1.27)))
     )
-    (property "Footprint" "" (at 284.48 135.89 0)
+    (property "Footprint" "" (at 284.48 137.16 0)
       (effects (font (size 1.27 1.27)) hide)
     )
-    (property "Datasheet" "" (at 284.48 135.89 0)
+    (property "Datasheet" "" (at 284.48 137.16 0)
       (effects (font (size 1.27 1.27)) hide)
     )
