File: TKL/TKL/TKL.kicad_sch (KiCad schematic)
At the start: 2 parts, among them U90 YAAJ_WeAct_BlackPill_Part_Lik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

Commit message: more finishing touches
Parts:
- added J1: Conn_01x02_Socket, Connector_PinHeader_2.00mm:PinHeader_1x02_P2.00mm_Vertical, symbol Connector:Conn_01x02_Socket
- U90: symbol YAAJ_WeAct_BlackPill_Part_Like_SWD_Breakout:YAAJ_WeAct_BlackPill_Part_Like_SWD_Breakout -> YAAJ_WeAct_BlackPill_Part_Like:YAAJ_WeAct_BlackPill_Part_Like
- USB1: footprint Type-C:HRO-TYPE-C-31-M-12-Assembly -> Type-C:USB_C_GCT_USB4085; symbol Type-C:HRO-TYPE-C-31-M-12 -> Type-C:12401598E4#2A
Connections:
- net CIN: now also U90.34 (PB0); no longer U90.30 (PA4)
- net COUT: now also J1.1 (Pin_1)
- net D+: now also USB1.B6 (D+); no longer USB1.6 (DP1)
- net D-: now also USB1.B7 (D-); no longer USB1.7 (DN1)
- net DIN: now also U90.33 (PA7); no longer U90.29 (PA3)
- net DOUT: now also J1.2 (Pin_2)
- net GND: now also USB1.A1 (GND), USB1.A12 (GND), USB1.B1 (GND), USB1.B12 (GND), USB1.S1 (Shell1), USB1.S2 (Shell2), USB1.S3 (Shell3), USB1.S4 (Shell4); no longer USB1.1 (GND), USB1.12 (GND), USB1.13 (SHIELD)
- net VCC: now also USB1.A4 (VBUS), USB1.A9 (VBUS), USB1.B4 (VBUS), USB1.B9 (VBUS); no longer USB1.11 (VBUS), USB1.2 (VBUS)

Commit message: fixed tkl schematic
Parts:
- added R1: 4.7kOhm, Resistor_THT:R_Axial_DIN0204_L3.6mm_D1.6mm_P7.62mm_Horizontal, symbol PCM_Resistor_AKL:R_0201
- added R2, R3: 10Ohm, Resistor_THT:R_Axial_DIN0204_L3.6mm_D1.6mm_P7.62mm_Horizontal, symbol PCM_Resistor_AKL:R_0201
- added R4: 390Ohm, Resistor_THT:R_Axial_DIN0204_L3.6mm_D1.6mm_P7.62mm_Horizontal, symbol PCM_Resistor_AKL:R_0201
Connections:
- net Col12: now also U90.32 (PA6); no longer U90.6 (PA9)
- net D+: now also USB1.A6 (D+), R3.2; no longer U90.9 (PA12)
- net D-: now also USB1.A7 (D-), R2.2; no longer U90.8 (PA11)
- net GND: now also R4.2
- net Row5: now also U90.31 (PA5); no longer U90.36 (PB2)
- net VCC: now also U90.18 (5V)
- net at USB1.B5 (CC2): now also R1.1
- new net: R1.2, R4.1
- new net: R2.1, U90.8 (PA11)
- new net: R3.1, U90.9 (PA12)
Changed lines of the file:
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@@
+    (stroke (width 0) (type default))
+  )
+  (wire (pts (xy 172.72 92.71) (xy 182.88 92.71))
     (stroke (width 0) (type default))
   )
@@
     (stroke (width 0) (type default))
   )
+  (wire (pts (xy 172.72 95.25) (xy 182.88 95.25))
+    (stroke (width 0) (type default))
+  )
   (wire (pts (xy 41.91 142.24) (xy 41.91 144.78))
     (stroke (width 0) (type default))
@@
     (stroke (width 0) (type default))
   )
+  (wire (pts (xy 41.91 109.22) (xy 49.53 109.22))
+    (stroke (width 0) (type default))
+  )
   (wire (pts (xy 177.8 120.65) (xy 182.88 120.65))
     (stroke (width 0) (type default))
@@
     )
   )
-  (global_label "Col12" (shape input) (at 182.88 87.63 180) (fields_autoplaced)
-    (effects (font (size 1.27 1.27)) (justify right))
-    (property "Intersheetrefs" "${INTERSHEET_REFS}" (at 175.1252 87.63 0)
-      (effects (font (size 1.27 1.27)) (justify right) hide)
+  (global_label "Col12" (shape input) (at 223.52 95.25 0) (fields_autoplaced)
+    (effects (font (size 1.27 1.27)) (justify left))
+    (property "Intersheetrefs" "${INTERSHEET_REFS}" (at 231.2748 95.25 0)
+      (effects (font (size 1.27 1.27)) (justify left) hide)
     )
   )
@@
     )
   )
+  (global_label "VCC" (shape input) (at 182.88 118.11 180) (fields_autoplaced)
+    (effects (font (size 1.27 1.27)) (justify right))
+    (property "Intersheetrefs" "${INTERSHEET_REFS}" (at 176.9998 118.11 0)
+      (effects (font (size 1.27 1.27)) (justify right) hide)
+    )
+  )
   (global_label "Col16" (shape input) (at 223.52 110.49 0) (fields_autoplaced)
     (effects (font (size 1.27 1.27)) (justify left))
@@
     )
   )
-  (global_label "D-" (shape input) (at 182.88 92.71 180) (fields_autoplaced)
-    (effects (font (size 1.27 1.27)) (justify right))
-    (property "Intersheetrefs" "${INTERSHEET_REFS}" (at 177.786 92.71 0)
+  (global_label "D-" (shape input) (at 165.1 92.71 180) (fields_autoplaced)
+    (effects (font (size 1.27 1.27)) (justify right))
+    (property "Intersheetrefs" "${INTERSHEET_REFS}" (at 160.006 92.71 0)
       (effects (font (size 1.27 1.27)) (justify right) hide)
     )
@@
     )
   )
-  (global_label "D+" (shape input) (at 182.88 95.25 180) (fields_autoplaced)
-    (effects (font (size 1.27 1.27)) (justify right))
-    (property "Intersheetrefs" "${INTERSHEET_REFS}" (at 177.786 95.25 0)
+  (global_label "D+" (shape input) (at 165.1 95.25 180) (fields_autoplaced)
+    (effects (font (size 1.27 1.27)) (justify right))
+    (property "Intersheetrefs" "${INTERSHEET_REFS}" (at 160.006 95.25 0)
       (effects (font (size 1.27 1.27)) (justify right) hide)
     )
@@
     )
   )
+  (global_label "D+" (shape input) (at 13.97 139.7 180) (fields_autoplaced)
+    (effects (font (size 1.27 1.27)) (justify right))
+    (property "Intersheetrefs" "${INTERSHEET_REFS}" (at 8.876 139.7 0)
+      (effects (font (size 1.27 1.27)) (justify right) hide)
+    )
+  )
   (global_label "Col11" (shape input) (at 87.63 68.58 0)
     (effects (font (size 1.27 1.27)) (justify left))
@@
     )
   )
-  (global_label "Row5" (shape input) (at 223.52 85.09 0) (fields_autoplaced)
-    (effects (font (size 1.27 1.27)) (justify left))
-    (property "Intersheetrefs" "${INTERSHEET_REFS}" (at 230.7306 85.09 0)
+  (global_label "Row5" (shape input) (at 223.52 97.79 0) (fields_autoplaced)
+    (effects (font (size 1.27 1.27)) (justify left))
+    (property "Intersheetrefs" "${INTERSHEET_REFS}" (at 230.7306 97.79 0)
       (effects (font (size 1.27 1.27)) (justify left) hide)
     )
@@
     )
   )
+  (global_label "D-" (shape input) (at 13.97 144.78 180) (fields_autoplaced)
+    (effects (font (size 1.27 1.27)) (justify right))
+    (property "Intersheetrefs" "${INTERSHEET_REFS}" (at 8.876 144.78 0)
+      (effects (font (size 1.27 1.27)) (justify right) hide)
+    )
+  )
   (global_label "Col10" (shape input) (at 68.58 35.56 180)
     (effects (font (size 1.27 1.27)) (justify right))
@@
     (property "Intersheetrefs" "${INTERSHEET_REFS}" (at 46.99 72.39 0)
       (effects (font (size 1.27 1.27)) hide)
+    )
+  )
+  (symbol (lib_id "power:GND") (at 49.53 124.46 0) (unit 1)
+    (in_bom yes) (on_board yes) (dnp no) (fields_autoplaced)
+    (property "Reference" "#PWR05" (at 49.53 130.81 0)
+      (effects (font (size 1.27 1.27)) hide)
+    )
+    (property "Value" "GND" (at 49.53 129.54 0)
+      (effects (font (size 1.27 1.27)))
+    )
+    (property "Footprint" "" (at 49.53 124.46 0)
+      (effects (font (size 1.27 1.27)) hide)
+    )
+    (property "Datasheet" "" (at 49.53 124.46 0)
+      (effects (font (size 1.27 1.27)) hide)
+    )
+    (pin "1")
+    (instances
+      (project "TKL"
+        (path "/b6c31d5e-0d78-456c-86e2-27aefb486f34"
+          (reference "#PWR05") (unit 1)
+        )
+      )
     )
   )
@@
         (path "/b6c31d5e-0d78-456c-86e2-27aefb486f34"
           (reference "#PWR04") (unit 1)
+        )
+      )
+    )
+  )
+  (symbol (lib_id "PCM_Resistor_AKL:R_0201") (at 49.53 113.03 0) (unit 1)
+    (in_bom yes) (on_board yes) (dnp no) (fields_autoplaced)
+    (property "Reference" "R1" (at 52.07 112.395 0)
+      (effects (font (size 1.27 1.27)) (justify left))
+    )
+    (property "Value" "4.7kOhm" (at 52.07 114.935 0)
+      (effects (font (size 1.27 1.27)) (justify left))
+    )
+    (property "Footprint" "Resistor_THT:R_Axial_DIN0204_L3.6mm_D1.6mm_P7.62mm_Horizontal" (at 49.53 124.46 0)
+      (effects (font (size 1.27 1.27)) hide)
+    )
+    (property "Datasheet" "~" (at 49.53 113.03 0)
+      (effects (font (size 1.27 1.27)) hide)
+    )
+    (pin "1")
+    (pin "2")
+    (instances
+      (project "TKL"
+        (path "/b6c31d5e-0d78-456c-86e2-27aefb486f34"
+          (reference "R1") (unit 1)
         )
       )
@@
         )
       )
+    )
+  )
+  (symbol (lib_id "PCM_Resistor_AKL:R_0201") (at 49.53 120.65 0) (unit 1)
+    (in_bom yes) (on_board yes) (dnp no) (fields_autoplaced)
+    (property "Reference" "R4" (at 52.07 120.015 0)
+      (effects (font (size 1.27 1.27)) (justify left))
+    )
+    (property "Value" "390Ohm" (at 52.07 122.555 0)
+      (effects (font (size 1.27 1.27)) (justify left))
+    )
+    (property "Footprint" "Resistor_THT:R_Axial_DIN0204_L3.6mm_D1.6mm_P7.62mm_Horizontal" (at 49.53 132.08 0)
+      (effects (font (size 1.27 1.27)) hide)
+    )
+    (property "Datasheet" "~" (at 49.53 120.65 0)
+      (effects (font (size 1.27 1.27)) hide)
+    )
+    (pin "1")
+    (pin "2")
+    (instances
+      (project "TKL"
+        (path "/b6c31d5e-0d78-456c-86e2-27aefb486f34"
+          (reference "R4") (unit 1)
+        )
+      )
+    )
+  )
+  (symbol (lib_id "PCM_Resistor_AKL:R_0201") (at 168.91 92.71 270) (unit 1)
+    (in_bom yes) (on_board yes) (dnp no) (fields_autoplaced)
+    (property "Reference" "R2" (at 168.91 87.63 90)
+      (effects (font (size 1.27 1.27)))
+    )
+    (property "Value" "10Ohm" (at 168.91 90.17 90)
+      (effects (font (size 1.27 1.27)))
+    )
+    (property "Footprint" "Resistor_THT:R_Axial_DIN0204_L3.6mm_D1.6mm_P7.62mm_Horizontal" (at 157.48 92.71 0)
+      (effects (font (size 1.27 1.27)) hide)
+    )
+    (property "Datasheet" "~" (at 168.91 92.71 0)
+      (effects (font (size 1.27 1.27)) hide)
+    )
+    (pin "1")
+    (pin "2")
+    (instances
+      (project "TKL"
+        (path "/b6c31d5e-0d78-456c-86e2-27aefb486f34"
+          (reference "R2") (unit 1)
+        )
+      )
+    )
+  )
+  (symbol (lib_id "PCM_Resistor_AKL:R_0201") (at 168.91 95.25 270) (unit 1)
+    (in_bom yes) (on_board yes) (dnp no)
+    (property "Reference" "R3" (at 168.91 99.695 90)
+      (effects (font (size 1.27 1.27)))
+    )
+    (property "Value" "10Ohm" (at 168.91 97.79 90)
+      (effects (font (size 1.27 1.27)))
+    )
+    (property "Footprint" "Resistor_THT:R_Axial_DIN0204_L3.6mm_D1.6mm_P7.62mm_Horizontal" (at 157.48 95.25 0)
+      (effects (font (size 1.27 1.27)) hide)
+    )
+    (property "Datasheet" "~" (at 168.91 95.25 0)
+      (effects (font (size 1.27 1.27)) hide)
+    )
+    (pin "1")
+    (pin "2")
+    (instances
+      (project "TKL"
+        (path "/b6c31d5e-0d78-456c-86e2-27aefb486f34"
+          (reference "R3") (unit 1)
+        )
+      )

Commit message: temp
Parts:
- added D88: BA595, Diode_SMD_AKL:D_SOD-323, symbol PCM_Diode_AKL:BA595
- added U91: STM32F401RETx, Package_QFP:LQFP-64_10x10mm_P0.5mm, symbol MCU_ST_STM32F4:STM32F401RETx
Connections:
- new net: U91.18 (VSS), U91.31 (VSS), U91.47 (VSS), U91.63 (VSS)
Changed lines of the file:
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@@
+    )
+  )
+  (symbol (lib_id "PCM_Diode_AKL:BA595") (at 113.03 132.08 0) (unit 1)
+    (in_bom yes) (on_board yes) (dnp no) (fields_autoplaced)
+    (property "Reference" "D88" (at 113.03 127 0)
+      (effects (font (size 1.27 1.27)))
+    )
+    (property "Value" "BA595" (at 113.03 129.54 0)
+      (effects (font (size 1.27 1.27)))
+    )
+    (property "Footprint" "Diode_SMD_AKL:D_SOD-323" (at 113.03 132.08 0)
+      (effects (font (size 1.27 1.27)) hide)
+    )
+    (property "Datasheet" "https://www.infineon.com/dgdl/Infineon-BA595_BA885_BA895SERIES-DS-v01_01-en.pdf?fileId=db3a304314dca3890114fdf44fbb09fe" (at 113.03 132.08 0)
+      (effects (font (size 1.27 1.27)) hide)
+    )
+    (pin "1")
+    (pin "2")
+    (instances
+      (project "TKL"
+        (path "/b6c31d5e-0d78-456c-86e2-27aefb486f34"
+          (reference "D88") (unit 1)
+        )
+      )
     )
   )
@@
         )
       )
+    )
+  )
+  (symbol (lib_id "MCU_ST_STM32F4:STM32F401RETx") (at 83.82 140.97 0) (unit 1)
+    (in_bom yes) (on_board yes) (dnp no) (fields_autoplaced)
+    (property "Reference" "U91" (at 88.3159 186.69 0)
+      (effects (font (size 1.27 1.27)) (justify left))
+    )
+    (property "Value" "STM32F401RETx" (at 88.3159 189.23 0)
+      (effects (font (size 1.27 1.27)) (justify left))
+    )
+    (property "Footprint" "Package_QFP:LQFP-64_10x10mm_P0.5mm" (at 71.12 184.15 0)
+      (effects (font (size 1.27 1.27)) (justify right) hide)
+    )
+    (property "Datasheet" "https://www.st.com/resource/en/datasheet/stm32f401re.pdf" (at 83.82 140.97 0)
+      (effects (font (size 1.27 1.27)) hide)
+    )
+    (pin "1")
+    (pin "10")
+    (pin "11")
+    (pin "12")
+    (pin "13")
+    (pin "14")
+    (pin "15")
+    (pin "16")
+    (pin "17")
+    (pin "18")
+    (pin "19")
+    (pin "2")
+    (pin "20")
+    (pin "21")
+    (pin "22")
+    (pin "23")
+    (pin "24")
+    (pin "25")
+    (pin "26")
+    (pin "27")
+    (pin "28")
+    (pin "29")
+    (pin "3")
+    (pin "30")
+    (pin "31")
+    (pin "32")
+    (pin "33")
+    (pin "34")
+    (pin "35")
+    (pin "36")
+    (pin "37")
+    (pin "38")
+    (pin "39")
+    (pin "4")
+    (pin "40")
+    (pin "41")
+    (pin "42")
+    (pin "43")
+    (pin "44")
+    (pin "45")
+    (pin "46")
+    (pin "47")
+    (pin "48")
+    (pin "49")
+    (pin "5")
+    (pin "50")
+    (pin "51")
+    (pin "52")
+    (pin "53")
+    (pin "54")
+    (pin "55")
+    (pin "56")
+    (pin "57")
+    (pin "58")
+    (pin "59")
+    (pin "6")
+    (pin "60")
+    (pin "61")
+    (pin "62")
+    (pin "63")
+    (pin "64")
+    (pin "7")
+    (pin "8")
+    (pin "9")
+    (instances
+      (project "TKL"
+        (path "/b6c31d5e-0d78-456c-86e2-27aefb486f34"
+          (reference "U91") (unit 1)
+        )
+      )
