File: prototypepcb/prototype.sch (KiCad schematic (older format))
At the start: 11 parts

Commit message: prototype pcb
Parts:
- added D? (x4): D_Small, symbol Device:D_Small
- added D? (x4): WS2812B, LED_SMD:LED_WS2812B_PLCC4_5.0x5.0mm_P3.2mm, symbol LED:WS2812B
- added MX? (x4): MX-NoLED, symbol MX_Alps_Hybrid:MX-NoLED
Connections:
- net +5V: now also D?.1 (VDD), D?.1 (VDD), D?.1 (VDD), D?.1 (VDD)
- net GND: now also D?.3 (VSS), D?.3 (VSS), D?.3 (VSS), D?.3 (VSS)
- net UGRGBDATA: now reaches U?.17 (PC2)
- net RGBDATA: now reaches U?.32 (PA7)
- net RGBDATA: now also D?.4 (DIN)
- net Row1: now reaches U?.35 (PB0)
- net Row1: now also D?.1 (K), D?.1 (K)
- net Col0: now reaches U?.36 (PB1)
- net Col0: now also MX?.1 (COL), MX?.1 (COL)
- net Col1: now reaches U?.37 (PB2)
- net Col1: now also MX?.1 (COL), MX?.1 (COL)
- net Row0: now reaches U?.89 (PB3)
- net Row0: now also D?.1 (K), D?.1 (K)
- new net: D?.2 (A), MX?.2 (ROW) (x4)
- new net: D?.2 (DOUT), D?.4 (DIN) (x3)
